File: WLED Controller.kicad_pcb (KiCad board)
At the start: 2 copper layers, 100 x 100 mm, 77 parts, among them J1 Power, J2 LED1, J3 LED1, J4 LED1, J5 AudioJack4, J6 LED1, J7 MD0, J8 MD1, K1 SANYOU_SRD_Form_C, Q1 AOD403, Q2 BC548, U1 74AHCT125, U2 AMS1117-3.3, U3 PCM1808PWR

Commit message: Added PDF and BOM.
Parts:
- moved C10 50.3 mm to (167.1, 81.4)
- moved C17 50.3 mm to (167.1, 96.6)
- moved C18 50.3 mm to (132.3, 143.3)
- moved C19 50.3 mm to (132.3, 140.2)
- moved C24 50.3 mm to (167.1, 111.8)
- moved C5 50.3 mm to (140.2, 72.6)
- moved C7 50.3 mm to (167.1, 66.2)
- moved D3 50.3 mm to (137.9, 55.9)
- moved DZ1 50.3 mm to (139.8, 77.5)
- moved F2 50.3 mm to (182.1, 66.0)
- moved F3 50.3 mm to (182.2, 81.3)
- moved F4 50.3 mm to (182.1, 96.5)
- moved F5 50.3 mm to (182.1, 111.8)
- moved G*** 50.3 mm to (135.3, 102.0)
- moved G*** 50.3 mm to (147.3, 104.0)
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Routing:
- net Net-(A1-ADC2_CH4/D13): track 13.4 -> 26.9 mm
- net Net-(D2-A): track 0.00 -> 6.85 mm
- net Net-(D1-A): track 0.00 -> 6.69 mm
- net Net-(A1-ADC2_CH6/D14): track 22.2 -> 27.7 mm
- net Net-(U3-VREF): track 7.12 -> 11.6 mm
- net +3.3V_D: track 61.6 -> 66.0 mm
- net +5V_D: track 179.8 -> 184.2 mm
- net Net-(J7-Pad2): track 8.02 -> 8.77 mm
Other:
- board text added: "©2025 Marc Schöndorf"

Commit message: Switched to 38pin ESP32 DevKit. Optimizations.
Parts:
- removed A1: ESP32_DevKit_V1_DOIT_30GPIOs, PCM_SL_Development_Boards:DOIT_ESP32_DEVKIT_30Pins
- removed J7: MD0, Connector_PinHeader_2.54mm:PinHeader_1x03_P2.54mm_Vertical
- removed J8: MD1, Connector_PinHeader_2.54mm:PinHeader_1x03_P2.54mm_Vertical
- added JP1: MD0, Jumper:SolderJumper-3_P1.3mm_Bridged12_Pad1.0x1.5mm, F.Cu at (138.7, 128.0)
- added JP2: MD1, Jumper:SolderJumper-3_P1.3mm_Bridged12_Pad1.0x1.5mm, F.Cu at (134.9, 128.0)
- added U2: ESP32-DevKitC, PCM_Espressif:ESP32-DevKitC, F.Cu at (150.5, 90.9)
- renumbered R3 to R2, R5 to R3, R6 to R4, R2 to R5, R4 to R6, U2 to U3, U3 to U4, U4 to U5
Connections:
- U5 pad 4: MIC_LR -> GND
Routing:
- net MIC_WS: track 0.00 -> 67.3 mm
- net MIC_SCK: track 0.00 -> 66.6 mm
- net MIC_SD: track 0.00 -> 63.5 mm
- net MCK: track 29.9 -> 57.1 mm
- net +3.3V_D: track 66.0 -> 80.5 mm
- net DOUT: track 33.9 -> 25.5 mm
- net Net-(R4-Pad1): track 27.0 -> 34.0 mm
- net +5V_D: track 184.2 -> 190.4 mm
- net Net-(U2-MTCK/GPIO13/ADC2_CH4): track 26.9 -> 21.2 mm
- net BCK: track 34.7 -> 30.3 mm
- net Net-(JP1-C): track 8.77 -> 4.37 mm
- net GND: track 63.9 -> 67.6 mm, vias 11 -> 194
- net Net-(R8-Pad1): track 41.2 -> 45.0 mm
- net DATA3: track 25.9 -> 23.5 mm
- net DATA2: track 36.8 -> 34.5 mm
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Other:
- board text added: "Audio pins"
- board text added: "MD0"
- board text added: "MD1"
- board text added: "MICROPHONE SD: GPIO 19 WS: GPIO 17 SCK: GPIO 18"
- board text added: "PCM1808 SD: GPIO 22 WS: GPIO 23 SCK: GPIO 21 MCLK: GPIO 0"
- board text removed: "+MD0-"
- board text removed: "+MD1-"
