File: WLED Controller.kicad_sch (KiCad schematic)
At the start: 73 parts, among them J1 Power, J2 LED1, J3 LED1, J4 LED1, J5 AudioJack4, J6 LED1, J7 MD0, J8 MD1, K1 SANYOU_SRD_Form_C, Q1 AOD403, Q2 BC548, U1 74AHCT125, U2 AMS1117-3.3, U3 PCM1808PWR

Commit message: Added PDF and BOM.
Other:
- company: Marc Schöndorf -> (C) 2025 Marc Schöndorf
Changed lines of the file:
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@@
 		(date "2025-01-20")
 		(rev "1.0.0")
-		(company "Marc Schöndorf")
+		(company "(C) 2025 Marc Schöndorf")
 	)
 	(junction

Commit message: Switched to 38pin ESP32 DevKit. Optimizations.
Parts:
- removed A1: ESP32_DevKit_V1_DOIT_30GPIOs, PCM_SL_Development_Boards:DOIT_ESP32_DEVKIT_30Pins, symbol PCM_SL_Development_Board:ESP32_DevKit_V1_DOIT_30GPIOs
- removed J7: MD0, Connector_PinHeader_2.54mm:PinHeader_1x03_P2.54mm_Vertical, symbol PCM_SL_Pin_Headers:PINHD_1x3_Male
- removed J8: MD1, Connector_PinHeader_2.54mm:PinHeader_1x03_P2.54mm_Vertical, symbol PCM_SL_Pin_Headers:PINHD_1x3_Male
- added JP1: MD0, Jumper:SolderJumper-3_P1.3mm_Bridged12_Pad1.0x1.5mm, symbol Jumper:SolderJumper_3_Bridged12
- added JP2: MD1, Jumper:SolderJumper-3_P1.3mm_Bridged12_Pad1.0x1.5mm, symbol Jumper:SolderJumper_3_Bridged12
- added U2: ESP32-DevKitC, PCM_Espressif:ESP32-DevKitC, symbol PCM_Espressif:ESP32-DevKitC
- renumbered R3 to R2, R5 to R3, R6 to R4, R2 to R5, R4 to R6, U2 to U3, U3 to U4, U4 to U5
Connections:
- net MIC_LR is gone; now on net GND: U5.4 (L/R)
- net +3.3V_D: now also JP1.3 (B), JP2.3 (B)
- net +5V_D: now also U2.19 (5V)
- net BCK: now also U2.33 (GPIO21)
- net DATA1: now also U2.10 (DAC_2/ADC2_CH9/GPIO26)
- net DATA2: now also U2.9 (DAC_1/ADC2_CH8/GPIO25)
- net DATA3: now also U2.8 (32K_XN/GPIO33/ADC1_CH5)
- net DATA4: now also U2.7 (32K_XP/GPIO32/ADC1_CH4)
- net DOUT: now also U2.36 (GPIO22)
- net GND: now also JP1.1 (A), JP2.1 (A), U2.14 (GND), U2.32 (GND), U2.38 (GND)
- net LRCK: now also U2.37 (GPIO23)
- net MCK: now also U2.25 (GPIO0/BOOT/ADC2_CH1)
- net MIC_SCK: now also U2.30 (GPIO18)
- net MIC_SD: now also U2.31 (GPIO19)
- net MIC_WS: now also U2.28 (GPIO17)
- net RELAY_CTRL: now also U2.11 (ADC2_CH7/GPIO27)
- net at R13.1: now also JP2.2 (C)
- net at R11.2: now also JP1.2 (C)
- net at R5.1: now also U2.15 (MTCK/GPIO13/ADC2_CH4)
- net at R6.2: now also U2.12 (MTMS/GPIO14/ADC2_CH6)
- no-connect marks 11 -> 18
Other:
- moved on the sheet: D1, D2, R5, R6

Commit message: Switched relay driver to MOSFET. Optimizations.
Parts:
- removed Q2: BC548, PCM_Package_TO_SOT_THT_AKL:TO-92_Inline_Wide_CBE, symbol PCM_Transistor_BJT_AKL:BC548
- added Q2: IRLL2705, PCM_Package_TO_SOT_SMD_AKL:SOT-223-3_TabPin2, symbol PCM_Transistor_MOSFET_AKL:IRLL2705
- added R14: 10k, PCM_Resistor_SMD_AKL:R_1206_3216Metric, symbol PCM_Resistor_AKL:R_1206
- renumbered R14 to R15
Connections:
- net GND: now also Q2.3 (S), R14.2
- net RELAY_CTRL: now also R14.1
- net at D3.2 (A), K1.2: now also Q2.2 (D)
- net at R12.1: now also Q2.1 (G)
Other:
- moved on the sheet: R12

Commit message: Optimizations
Parts:
- added JP1: R2 GND, Jumper:SolderJumper-3_P1.3mm_Bridged12_Pad1.0x1.5mm, symbol Jumper:SolderJumper_3_Bridged12
- renumbered C21 to C20, C22 to C21, C20 to C22, JP1 to JP2, JP2 to JP3
Connections:
- net GND: now also JP1.1 (A); no longer J5.R2
- new net: J5.R2, JP1.2 (C)
Other:
- moved on the sheet: C18, C19, C20, C21, R10, R9
